File: Encoder_Breakout.kicad_pcb (KiCad board)
At the start: 2 copper layers, 29.2 x 24.1 mm, 4 parts, among them J1 Conn_01x03, J2 Conn_02x07_Odd_Even, J3 Conn_01x02, J4 Conn_01x02

Commit message: PCB changes and add kibot
Signed-off-by: Colin <cfinn68916@gmail.com>
Parts:
- removed J3, J4: Conn_01x02, Connector_PinSocket_2.54mm:PinSocket_1x02_P2.54mm_Vertical
- added J5: 5-104935-3, footprints:CONN_5-104935-3_TYCO, F.Cu at (142.3, 90.2)
- added J6: 5-104363-1, footprints:CONN_5-104363-1_TYCO, F.Cu at (149.2, 102.2)
- J1: value Conn_01x03 -> 5-104363-1; footprint Connector_PinHeader_2.54mm:PinHeader_1x03_P2.54mm_Horizontal -> footprints:CONN_5-104363-1_TYCO
- moved J1 15.2 mm to (151.8, 76.0)
Connections:
- J1 pad 1: Net-(J1-Pin_1) -> Net-(J2-Pin_6)
- J1 pad 2: +3.3V -> GND
- J2 pad 5: Net-(J1-Pin_1) -> Net-(J2-Pin_5)
Routing:
- net GND: track 47.7 -> 68.8 mm
- net Net-(J2-Pin_5): track 0.00 -> 19.3 mm
- net Net-(J1-Pin_1): track 15.5 -> 0.00 mm
- net +3.3V: track 15.0 -> 18.7 mm
- net Net-(J2-Pin_6): track 16.8 -> 19.8 mm
- net Net-(J2-Pin_10): track 25.2 -> 22.9 mm
Other:
- board size 29.2 x 24.1 mm -> 35.6 x 33.7 mm
- board text added: "FRC Team 1716 Redbird Robotics"
- board text removed: "1716"
